Commit message: Barista urdf model has been complete

File: urdf/barista_robot_model.urdf (robot description, URDF)
Before this commit: robot barista_bot, 11 links, 10 joints
Links:
- added link hokuyo_laser_link; collision mesh filename=package://barista_robot_description/meshes/hokuyo_urg_04lx.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; visual mesh filename=package://barista_robot_description/meshes/hokuyo_urg_04lx.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
Joints:
- added joint barista_body_hokuyo_laser_joint: type fixed, parent barista_body, child hokuyo_laser_link, origin xyz=0 -0.0895 0.1726 rpy=0 0 0
- joint barista_body_barista_top_joint: origin xyz=0 0 0.4454 rpy=0 0 0 -> xyz=0 0 0.4376 rpy=0 0 0
- joint barista_body_standoff_rod_four_joint: origin xyz=-0.0895 -0.0895 0.2883 rpy=0 0 0 -> xyz=-0.0895 -0.0543 0.1726 rpy=0 0 0
- joint barista_body_standoff_rod_one_joint: origin xyz=0.0895 0.0895 0.2883 rpy=0 0 0 -> xyz=0.0895 0.0543 0.1726 rpy=0 0 0
- joint barista_body_standoff_rod_three_joint: origin xyz=-0.0895 0.0895 0.2883 rpy=0 0 0 -> xyz=-0.0895 0.0543 0.1726 rpy=0 0 0
- joint barista_body_standoff_rod_two_joint: origin xyz=0.0895 -0.0895 0.2883 rpy=0 0 0 -> xyz=0.0895 -0.0543 0.1726 rpy=0 0 0

Commit message: Gazebo plugins have been added to the urdf file which allows the barista bot to be controlled using the /cmd_vel topic.

File: urdf/barista_robot_model.urdf (robot description, URDF)
Before this commit: robot my_robot, 12 links, 11 joints
Links:
- link back_caster_wheel: mass 1.5 -> 0.5
- link front_caster_wheel: mass 1.5 -> 0.5
Joints:
- joint barista_body_back_caster_wheel_joint: axis (none) -> 1 0 0; origin xyz=0 -0.1198 0.0352 rpy=0 0 0 -> xyz=0 0.135 0.0352 rpy=0 0 0; type fixed -> continuous
- joint barista_body_front_caster_wheel_joint: axis (none) -> 1 0 0; origin xyz=0 0.1198 0.0352 rpy=0 0 0 -> xyz=0 -0.135 0.0352 rpy=0 0 0; type fixed -> continuous
